File: handheld_featherwing.kicad_pcb (KiCad board)
At the start: 2 copper layers, 0 parts

Commit message: Finish up rev1
Parts:
- added C1: 0.1uF, Capacitor_SMD:C_0603_1608Metric, F.Cu at (171.3, 99.3)
- added C10: 0.1uF, Capacitor_SMD:C_0603_1608Metric, F.Cu at (142.0, 93.9)
- added C11: 0.1uF, Capacitor_SMD:C_0603_1608Metric, F.Cu at (165.6, 94.2)
- added C12: 0.1uF, Capacitor_SMD:C_0603_1608Metric, F.Cu at (159.5, 103.5)
- added C2: 10uF, Capacitor_SMD:C_0603_1608Metric, F.Cu at (165.6, 107.4)
- added C3: 1uF, Capacitor_SMD:C_0603_1608Metric, F.Cu at (164.1, 107.4)
- added C4: 0.1uF, Capacitor_SMD:C_0603_1608Metric, F.Cu at (134.9, 83.1)
- added C5: 10uF, Capacitor_SMD:C_0603_1608Metric, F.Cu at (134.9, 86.1)
- added C6: 0.1uF, Capacitor_SMD:C_0603_1608Metric, F.Cu at (135.1, 94.4)
- added C7: 0.1uF, Capacitor_SMD:C_0603_1608Metric, F.Cu at (139.9, 99.7)
- added C8: 0.1uF, Capacitor_SMD:C_0603_1608Metric, F.Cu at (138.4, 99.7)
- added C9: 10uF, Capacitor_SMD:C_0603_1608Metric, F.Cu at (138.4, 96.6)
- added D1: WS2812B, LED_SMD:LED_WS2812B_PLCC4_5.0x5.0mm_P3.2mm, B.Cu at (120.8, 49.8)
- added D2: S1JHE, Diode_SMD:D_SOD-323, F.Cu at (126.8, 52.6)
- added D3: S1JHE, Diode_SMD:D_SOD-323, F.Cu at (126.8, 54.6)
- added G***: LOGO, Symbol:OSHW-Logo_11.4x12mm_SilkScreen, B.Cu at (139.0, 125.2)
- added G***: LOGO, Symbol:KiCad-Logo2_12mm_SilkScreen, B.Cu at (139.6, 73.5)
- added G***: LOGO, Symbols_Extra:SolderParty-Logo_14.6x13.5mm_SilkScreen, F.Cu at (152.4, 124.4)
- added J3: Micro_SD_Card_Det, Connector_Card_Extra:microSD_HC_Molex_104031-0811, F.Cu at (153.1, 56.1)
- added JP1: SB_CARD_CS, Jumper:SolderJumper-2_P1.3mm_Bridged_RoundedPad1.0x1.5mm, F.Cu at (162.4, 55.4)
- added JP2: SB_LCD_CS, Jumper:SolderJumper-2_P1.3mm_Bridged_RoundedPad1.0x1.5mm, F.Cu at (135.1, 100.4)
- added JP3: SB_LCD_DC, Jumper:SolderJumper-2_P1.3mm_Bridged_RoundedPad1.0x1.5mm, F.Cu at (135.1, 102.9)
- added JP4: SB_MIC_VDD, Jumper:SolderJumper-2_P1.3mm_Open_RoundedPad1.0x1.5mm, F.Cu at (154.3, 81.8)
- added JP5: SB_STM_CS, Jumper:SolderJumper-2_P1.3mm_Bridged_RoundedPad1.0x1.5mm, F.Cu at (135.1, 97.9)
- added JP6: SB_NEOPIXEL, Jumper:SolderJumper-2_P1.3mm_Bridged_RoundedPad1.0x1.5mm, F.Cu at (120.8, 53.9)
- added Q1: BSS138, Package_TO_SOT_SMD:SOT-23, F.Cu at (149.6, 80.5)
- added Q2: BSS138, Package_TO_SOT_SMD:SOT-23, F.Cu at (126.8, 57.6)
- added R1: 4.7K, Resistor_SMD:R_0603_1608Metric, F.Cu at (143.6, 93.9)
- added R2: 4.7K, Resistor_SMD:R_0603_1608Metric, F.Cu at (143.6, 99.7)
- added R3: 10K, Resistor_SMD:R_0603_1608Metric, F.Cu at (162.4, 58.0)
- added R4: 10K, Resistor_SMD:R_0603_1608Metric, F.Cu at (147.0, 80.5)
- added R5: 1K, Resistor_SMD:R_0603_1608Metric, F.Cu at (167.1, 107.4)
- added R6: 10K, Resistor_SMD:R_0603_1608Metric, F.Cu at (124.2, 57.6)
- added R7: 10R, Resistor_SMD:R_0603_1608Metric, F.Cu at (129.3, 57.6)
- added R8: 10K, Resistor_SMD:R_0603_1608Metric, F.Cu at (131.6, 99.5)
- added R9: 10K, Resistor_SMD:R_0603_1608Metric, F.Cu at (135.1, 95.9)
- added REF**: MountingHole_3.2mm_M3, MountingHole:MountingHole_3.2mm_M3, F.Cu at (112.2, 50.0)
- added REF**: MountingHole_3.2mm_M3, MountingHole:MountingHole_3.2mm_M3, F.Cu at (165.8, 142.4)
- added REF**: MountingHole_3.2mm_M3, MountingHole:MountingHole_3.2mm_M3, F.Cu at (112.2, 142.4)
- added REF**: Fiducial_0.5mm_Dia_1mm_Outer, Fiducial:Fiducial_0.5mm_Dia_1mm_Outer, B.Cu at (137.1, 76.2)
- added REF**: Fiducial_0.5mm_Dia_1mm_Outer, Fiducial:Fiducial_0.5mm_Dia_1mm_Outer, B.Cu at (139.0, 123.7)
- added REF**: MountingHole_3.2mm_M3, MountingHole:MountingHole_3.2mm_M3, F.Cu at (165.8, 50.0)
- added SW1: SW_EN, Button_Switch_SMD:SW_SPDT_PCM12, F.Cu at (130.5, 48.1)
- added SW2: SW_RIGHT1, Button_Switch_SMD_Extra:RMT-CZ66, B.Cu at (112.9, 104.0)
- added SW3: SW_LEFT1, Button_Switch_SMD_Extra:RMT-CZ66, B.Cu at (165.1, 104.0)
- added SW4: SW_RIGHT2, Button_Switch_SMD_Extra:RMT-CZ66, B.Cu at (126.2, 104.0)
- added SW5: SW_LEFT2, Button_Switch_SMD_Extra:RMT-CZ66, B.Cu at (151.8, 104.0)
- added TP1: TP_MIC, TestPoint:TestPoint_Pad_D3.0mm, F.Cu at (154.2, 85.4)
- added TP10: TP_KBD_GND, TestPoint:TestPoint_Pad_D3.0mm, F.Cu at (162.0, 113.1)
- added TP2: TP_KBD_SWCLK, TestPoint:TestPoint_Pad_D3.0mm, F.Cu at (157.9, 113.1)
- added TP3: TP_KBD_SWDIO, TestPoint:TestPoint_Pad_D3.0mm, F.Cu at (166.1, 113.1)
- added TP4: TP_KBD_TX, TestPoint:TestPoint_Pad_D3.0mm, F.Cu at (164.9, 120.0)
- added TP5: TP_STM_INT, TestPoint:TestPoint_Pad_D3.0mm, F.Cu at (145.7, 117.2)
- added TP6: TP_MAG_DRDY, TestPoint:TestPoint_Pad_D3.0mm, F.Cu at (145.7, 109.0)
- added TP7: TP_MAG_INT, TestPoint:TestPoint_Pad_D3.0mm, F.Cu at (145.7, 113.1)
- added TP8: TP_ACCEL_INT, TestPoint:TestPoint_Pad_D3.0mm, F.Cu at (145.7, 104.9)
- added TP9: TP_KBD_3V, TestPoint:TestPoint_Pad_D3.0mm, F.Cu at (153.8, 113.1)
- added U1: 5-Way_Switch, Button_Switch_SMD_Extra:SF303GJ26, B.Cu at (139.0, 104.0)
- added U2: BBQ10KBD, Connector_Hirose_Extra:BM14B(0.8)-24DS-0.4V(53), F.Cu at (148.6, 88.0)
- added U3: LSM303C, Package_LGA:LGA-12_2x2mm_P0.5mm, F.Cu at (141.2, 96.8)
- added U4: ER-TFT02X, Connector_EastRising:ER-CON50HT-1, F.Cu at (128.4, 75.7)
- added U5: STMPE811, Package_DFN_QFN:QFN-16-1EP_3x3mm_P0.5mm_EP1.75x1.75mm, F.Cu at (130.7, 94.6)
- added U6: Adafruit_Feather_2X, Module_Extra:FeatherWing, F.Cu at (151.8, 71.5)
- added U7: ATSAMD20G16A, Package_DFN_QFN:QFN-48-1EP_7x7mm_P0.5mm_EP5.15x5.15mm, F.Cu at (164.9, 100.2)
- added U8: 74AHCT1G125, Package_TO_SOT_SMD:SOT-23-5, F.Cu at (120.8, 49.8)
Routing:
- net +3V3: track 0.00 -> 270.0 mm, vias 0 -> 17
- net /KBD_RESET: track 0.00 -> 129.3 mm, vias 0 -> 8
- net /CARD_MISO: track 0.00 -> 92.5 mm, vias 0 -> 3
- net GND: track 0.00 -> 88.9 mm, vias 0 -> 147
- net /CARD_MOSI: track 0.00 -> 82.5 mm, vias 0 -> 5
- net /CARD_CLK: track 0.00 -> 77.3 mm, vias 0 -> 2
- net /KBD_INT: track 0.00 -> 65.0 mm, vias 0 -> 4
- net /Keyboard/BTN_RIGHT1: track 0.00 -> 64.6 mm, vias 0 -> 1
- net /GPIO11: track 0.00 -> 62.0 mm, vias 0 -> 2
- net /GPIO10: track 0.00 -> 55.6 mm, vias 0 -> 2
- net /Keyboard/BTN_RIGHT2: track 0.00 -> 52.2 mm, vias 0 -> 1
- net VBUS: track 0.00 -> 51.8 mm, vias 0 -> 2
- net /EN: track 0.00 -> 50.7 mm, vias 0 -> 2
- net /ACCEL_SCL: track 0.00 -> 45.5 mm, vias 0 -> 2
- net /CARD_DET: track 0.00 -> 44.9 mm, vias 0 -> 2
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- added copper zone on B.Cu, net GND
- added copper zone on F.Cu, net GND
Other:
- board outline added: 68 x 100 mm
- rule trace_min: 0.2 -> 0.15
- rule via_min_size: 0.4 -> 0.55
- board text added: "3.3V"
- board text added: "@arturo182"
- board text added: "ACCEL INT"
- board text added: "CARD CS"
- board text added: "CLK"
- board text added: "GND"
- board text added: "GPIOs used: GPIO05: CARD CS GPIO06: STMP CS GPIO09: LCD CS GPIO10: LCD DC GPIO11: NEOPIX"
- board text added: "Handheld FeatherWing by arturo182 May 2019"
- board text added: "IO"
- board text added: "KBD IC SWD"
- board text added: "KBD TX"
- board text added: "MAG DRDY"
- board text added: "MAG INT"
- board text added: "MIC"
- board text added: "MIC EN"
- board text added: "NEOPIX"
- board text added: "STMP CS LCD CS LCD DC"
- board text added: "STMP INT"

Commit message: rev2
Parts:
- D2, D3: footprint Diode_SMD:D_SOD-323 -> Diode_SMD:D_SOD-323_HandSoldering
- REF** (x4): value MountingHole_3.2mm_M3 -> MountingHole_3.2mm_M3_with_paste; footprint MountingHole:MountingHole_3.2mm_M3 -> MountingHole_Extra:MountingHole_3.2mm_M3_with_paste
- U8: footprint Package_TO_SOT_SMD:SOT-23-5 -> Package_TO_SOT_SMD:SOT-353_SC-70-5
- moved D2 0.25 mm to (126.8, 52.4)
Connections:
- D1 pad 2: Net-(D1-Pad2) -> (no net)
- J3 pad 1: Net-(J3-Pad1) -> (no net)
- J3 pad 8: Net-(J3-Pad8) -> (no net)
- SW1 pad 1: Net-(SW1-Pad1) -> (no net)
- U4 pad 39: Net-(U4-Pad39) -> (no net)
- U7 pad 15: Net-(U7-Pad15) -> (no net)
- U7 pad 16: Net-(U7-Pad16) -> (no net)
- U7 pad 33: Net-(U7-Pad33) -> (no net)
- U7 pad 34: Net-(U7-Pad34) -> (no net)
- U7 pad 38: Net-(U7-Pad38) -> (no net)
- U7 pad 39: Net-(U7-Pad39) -> (no net)
- U7 pad 41: Net-(U7-Pad41) -> (no net)
- U7 pad 47: Net-(U7-Pad47) -> (no net)
- U7 pad 48: Net-(U7-Pad48) -> (no net)
- U7 pad 7: Net-(U7-Pad7) -> (no net)
Routing:
- net GND: track 88.9 -> 86.5 mm, vias 147 -> 143
- net VBUS: track 51.8 -> 50.0 mm
- net /GPIO11: track 62.0 -> 60.6 mm
- net Net-(U6-Pad16): track 5.04 -> 5.74 mm
- net /GPIO5: track 42.7 -> 43.3 mm
- net +3V3: track 270.0 -> 270.6 mm
- net +5V: track 15.5 -> 14.9 mm
Other:
- outline, holes or cut-outs redrawn
- board text added: "10"
- board text added: "11"
- board text added: "12"
- board text added: "13"
- board text added: "3V"
- board text added: "5"
- board text added: "6"
- board text added: "9"
- board text added: "@"
- board text added: "A0"
- board text added: "A1"
- board text added: "A2"
- board text added: "A3"
- board text added: "A4"
- board text added: "A5"
- board text added: "Aref"
- board text added: "BAT"
- board text added: "EN"
- board text added: "GPIOs: GPIO05: CARD CS GPIO06: STMP CS GPIO09: LCD CS GPIO10: LCD DC GPIO11: NEOPIXEL I2C: 0x1D - Accel 0x1E - Mag 0x1F - Keyboard"
- board text added: "Keyboard FeatherWing by arturo182 June 2019"
- board text added: "MI"
- board text added: "MISC"
- board text added: "MO"
- board text added: "NEOPIXEL"
- board text added: "OFF"
- board text added: "ON"
- board text added: "RST"
- board text added: "RX"
- board text added: "SCK"
- board text added: "SCL"
- board text added: "SDA"
- board text added: "TX"
- board text added: "USB"
- board text added: "arturo182"
- board text removed: "@arturo182"
- board text removed: "GPIOs used: GPIO05: CARD CS GPIO06: STMP CS GPIO09: LCD CS GPIO10: LCD DC GPIO11: NEOPIX"
- board text removed: "Handheld FeatherWing by arturo182 May 2019"
- board text removed: "NEOPIX"

Commit message: Rev 3
Parts:
- removed C10, C7, C8: 0.1uF, Capacitor_SMD:C_0603_1608Metric
- removed C9: 10uF, Capacitor_SMD:C_0603_1608Metric
- removed TP6: TP_MAG_DRDY, TestPoint:TestPoint_Pad_D3.0mm
- removed TP7: TP_MAG_INT, TestPoint:TestPoint_Pad_D3.0mm
- removed TP8: TP_ACCEL_INT, TestPoint:TestPoint_Pad_D3.0mm
- removed U3: LSM303C, Package_LGA:LGA-12_2x2mm_P0.5mm
- moved TP5 15.3 mm to (135.1, 106.2)
- moved R2 5.99 mm to (142.1, 93.9), turned to -90 degrees
Connections:
- net /ACCEL_SCL renamed /KBD_SCL
- net /ACCEL_SDA renamed /KBD_SDA
- D1 pad 2: (no net) -> Net-(D1-Pad2)
- J3 pad 1: (no net) -> Net-(J3-Pad1)
- J3 pad 8: (no net) -> Net-(J3-Pad8)
- SW1 pad 1: (no net) -> Net-(SW1-Pad1)
- U4 pad 39: (no net) -> Net-(U4-Pad39)
- U7 pad 15: (no net) -> Net-(U7-Pad15)
- U7 pad 16: (no net) -> Net-(U7-Pad16)
- U7 pad 33: (no net) -> Net-(U7-Pad33)
- U7 pad 34: (no net) -> Net-(U7-Pad34)
- U7 pad 38: (no net) -> Net-(U7-Pad38)
- U7 pad 39: (no net) -> Net-(U7-Pad39)
- U7 pad 41: (no net) -> Net-(U7-Pad41)
- U7 pad 47: (no net) -> Net-(U7-Pad47)
- U7 pad 48: (no net) -> Net-(U7-Pad48)
- U7 pad 7: (no net) -> Net-(U7-Pad7)
Routing:
- net Net-(TP7-Pad1): track 23.4 -> 0.00 mm, vias 2 -> 0
- net Net-(TP5-Pad1): track 33.5 -> 15.5 mm
- net Net-(TP6-Pad1): track 13.4 -> 0.00 mm
- net Net-(TP8-Pad1): track 10.2 -> 0.00 mm
- net +3V3: track 270.6 -> 262.6 mm
- net GND: track 86.5 -> 90.1 mm, vias 143 -> 141
- net /KBD_SDA: track 40.2 -> 37.9 mm
- net /GPIO10: track 55.6 -> 53.8 mm
- net Net-(C10-Pad1): track 1.58 -> 0.00 mm
- net /GPIO9: track 43.2 -> 41.9 mm
- net /KBD_SCL: track 45.8 -> 44.7 mm
- net /GPIO6: track 40.0 -> 39.2 mm
- net /CARD_MISO: track 92.5 -> 93.1 mm
Other:
- board text added: "GPIOs: D5: CARD CS D6: STMP CS D9: LCD CS D10: LCD DC D11: NEOPIXEL I2C: 0x1F - Keyboard"
- board text added: "Keyboard FeatherWing by arturo182 March 2020"
- board text added: "LCD CS"
- board text added: "LCD DC"
- board text added: "STMP CS"
- board text removed: "ACCEL INT"
- board text removed: "GPIOs: GPIO05: CARD CS GPIO06: STMP CS GPIO09: LCD CS GPIO10: LCD DC GPIO11: NEOPIXEL I2C: 0x1D - Accel 0x1E - Mag 0x1F - Keyboard"
- board text removed: "Keyboard FeatherWing by arturo182 June 2019"
- board text removed: "MAG DRDY"
- board text removed: "MAG INT"
- board text removed: "STMP CS LCD CS LCD DC"

Commit message: Rev 4!
Parts:
- added J7: Conn_Stemma_QT, Connector_JST:JST_SH_SM04B-SRSS-TB_1x04-1MP_P1.00mm_Horizontal, F.Cu at (108.3, 98.1)
- moved TP5 0.50 mm to (135.1, 106.7)
Routing:
- net /KBD_SDA: track 37.9 -> 83.4 mm
- net /KBD_SCL: track 44.7 -> 85.4 mm
- net +3V3: track 262.6 -> 280.6 mm, vias 17 -> 20
- net /KBD_RESET: track 129.5 -> 136.7 mm, vias 8 -> 6
- net /LCD_CS: track 39.9 -> 41.0 mm
- net /LCD_DC: track 43.9 -> 44.9 mm
- net /Keyboard/KBD_COL4: track 20.9 -> 20.0 mm
- net /Keyboard/KBD_ROW3: track 22.3 -> 21.4 mm
- net /Keyboard/KBD_ROW4: track 24.6 -> 23.7 mm
- net /Keyboard/KBD_ROW6: track 27.2 -> 26.4 mm
- net /Keyboard/KBD_COL5: track 23.3 -> 22.5 mm
- net /Keyboard/KBD_ROW5: track 25.8 -> 25.0 mm
- net /Keyboard/KBD_ROW7: track 30.4 -> 29.6 mm
- net Net-(TP5-Pad1): track 15.5 -> 16.1 mm
- net /CARD_MISO: track 93.1 -> 93.7 mm
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Other:
- board text added: "Qwiic STEMMA QT"
