File: handheld_featherwing.sch (KiCad schematic (older format))
At the start: 14 parts, among them J3 Micro_SD_Card_Det, SW1 SW_EN, U5 STMPE811, U6 Adafruit_Feather_2X

Commit message: Finish up rev1
Parts:
- added C10, C7, C8: 0.1uF, Capacitor_SMD:C_0603_1608Metric, symbol Device:C_Small
- added C9: 10uF, Capacitor_SMD:C_0603_1608Metric, symbol Device:C_Small
- added D1: WS2812B, LED_SMD:LED_WS2812B_PLCC4_5.0x5.0mm_P3.2mm, symbol LED:WS2812B
- added D2, D3: S1JHE, Diode_SMD:D_SOD-323, symbol Device:D_Schottky_Small
- added JP6: SB_NEOPIXEL, Jumper:SolderJumper-2_P1.3mm_Bridged_RoundedPad1.0x1.5mm, symbol Jumper:SolderJumper_2_Bridged
- added TP6: TP_MAG_DRDY, TestPoint:TestPoint_Pad_D3.0mm, symbol Connector:TestPoint
- added TP7: TP_MAG_INT, TestPoint:TestPoint_Pad_D3.0mm, symbol Connector:TestPoint
- added TP8: TP_ACCEL_INT, TestPoint:TestPoint_Pad_D3.0mm, symbol Connector:TestPoint
- added U3: LSM303C, Package_LGA:LGA-12_2x2mm_P0.5mm, symbol Sensor_Motion_Extra:LSM303C
- added U8: 74AHCT1G125, Package_TO_SOT_SMD:SOT-23-5, symbol 74xGxx:74AHCT1G125
- J3: footprint (none) -> Connector_Card_Extra:microSD_HC_Molex_104031-0811
- SW1: footprint (none) -> Button_Switch_SMD:SW_SPDT_PCM12
- U6: footprint (none) -> Module_Extra:FeatherWing
Connections:
- net +3V3: now also C7.1, C8.1, C9.1, U3.10 (VDDIO), U3.2 (CS_XL), U3.3 (CS_MAG), U3.9 (VDD)
- net +BATT: now also D3.2 (A)
- net GND: now also C10.2, C7.2, C8.2, C9.2, D1.3 (VSS), U3.6 (GND), U3.8 (GND), U8.1, U8.3 (GND)
- net GPIO11: now also JP6.1 (A)
- net VBUS: now also D2.2 (A)
- net KBD_SCL renamed ACCEL_SCL
- net ACCEL_SCL: now also U3.1 (SCL)
- net KBD_SDA renamed ACCEL_SDA
- net ACCEL_SDA: now also U3.4 (SDA)
- new net: TP6.1, U3.11 (DRDY_MAG)
- new net: TP8.1, U3.12 (INT_XL)
- new net: C10.1, U3.5 (C1)
- new net: TP7.1, U3.7 (INT_MAG)
- new net: D1.4 (DIN), U8.4
- new net +5V: D1.1 (VDD), D2.1 (K), D3.1 (K), U8.5 (VCC)
- new net NEOPIXEL: JP6.2 (B), U8.2
- no-connect marks 3 -> 4
Other:
- note removed: "ADD NEOPIXEL, YO!\n"
- moved on the sheet: JP1, JP2, JP3, JP5, R1, R2, SW1

Commit message: rev2
Parts:
- D2, D3: footprint Diode_SMD:D_SOD-323 -> Diode_SMD:D_SOD-323_HandSoldering
- U8: footprint Package_TO_SOT_SMD:SOT-23-5 -> Package_TO_SOT_SMD:SOT-353_SC-70-5
Changed lines of the file:
@@
 EESchema Schematic File Version 4
-LIBS:handheld_featherwing-cache
 EELAYER 29 0
 EELAYER END
@@
 Wire Wire Line
 	9050 3300 9100 3300
-$Comp
-L Jumper:SolderJumper_2_Bridged JP1
-U 1 1 5CDA97F7
-P 9250 3300
-F 0 "JP1" H 9250 3413 50  0000 C CNN
-F 1 "SB_CARD_CS" H 9250 3414 50  0001 C CNN
-F 2 "Jumper:SolderJumper-2_P1.3mm_Bridged_RoundedPad1.0x1.5mm" H 9250 3300 50  0001 C CNN
-F 3 "~" H 9250 3300 50  0001 C CNN
-	1    9250 3300
-	1    0    0    -1
-$EndComp
 Wire Wire Line
 	9400 3300 9450 3300
@@
 F 0 "U8" H 8750 1550 50  0000 C CNN
 F 1 "74AHCT1G125" H 8600 1200 50  0000 C CNN
-F 2 "Package_TO_SOT_SMD:SOT-23-5" H 8900 1400 50  0001 C CNN
+F 2 "Package_TO_SOT_SMD:SOT-353_SC-70-5" H 8900 1400 50  0001 C CNN
 F 3 "http://www.ti.com/lit/sg/scyt129e/scyt129e.pdf" H 8900 1400 50  0001 C CNN
 	1    8900 1400
@@
 F 0 "D2" H 9350 2150 50  0000 C CNN
 F 1 "S1JHE" H 9250 2086 50  0001 C CNN
-F 2 "Diode_SMD:D_SOD-323" V 9250 2200 50  0001 C CNN
+F 2 "Diode_SMD:D_SOD-323_HandSoldering" V 9250 2200 50  0001 C CNN
 F 3 "~" V 9250 2200 50  0001 C CNN
 	1    9250 2200
@@
 F 0 "D3" H 9350 2300 50  0000 C CNN
 F 1 "S1JHE" H 9250 2236 50  0001 C CNN
-F 2 "Diode_SMD:D_SOD-323" V 9250 2350 50  0001 C CNN
+F 2 "Diode_SMD:D_SOD-323_HandSoldering" V 9250 2350 50  0001 C CNN
 F 3 "~" V 9250 2350 50  0001 C CNN
 	1    9250 2350
@@
 	-1   0    0    1
 $EndComp
+$Comp
+L Jumper:SolderJumper_2_Bridged JP1
+U 1 1 5CDA97F7
+P 9250 3300
+F 0 "JP1" H 9250 3413 50  0000 C CNN
+F 1 "SB_CARD_CS" H 9250 3414 50  0001 C CNN
+F 2 "Jumper:SolderJumper-2_P1.3mm_Bridged_RoundedPad1.0x1.5mm" H 9250 3300 50  0001 C CNN
+F 3 "~" H 9250 3300 50  0001 C CNN
+	1    9250 3300
+	1    0    0    -1
+$EndComp
 $EndSCHEMATC

Commit message: Rev 3
Parts:
- removed C10, C7, C8: 0.1uF, Capacitor_SMD:C_0603_1608Metric, symbol Device:C_Small
- removed C9: 10uF, Capacitor_SMD:C_0603_1608Metric, symbol Device:C_Small
- removed TP6: TP_MAG_DRDY, TestPoint:TestPoint_Pad_D3.0mm, symbol Connector:TestPoint
- removed TP7: TP_MAG_INT, TestPoint:TestPoint_Pad_D3.0mm, symbol Connector:TestPoint
- removed TP8: TP_ACCEL_INT, TestPoint:TestPoint_Pad_D3.0mm, symbol Connector:TestPoint
- removed U3: LSM303C, Package_LGA:LGA-12_2x2mm_P0.5mm, symbol Sensor_Motion_Extra:LSM303C
Connections:
- net ACCEL_SCL renamed KBD_SCL
- net ACCEL_SDA renamed KBD_SDA
- no-connect marks 4 -> 5

Commit message: Rev 4!
Parts:
- added J7: Conn_Stemma_QT, Connector_JST:JST_SH_SM04B-SRSS-TB_1x04-1MP_P1.00mm_Horizontal, symbol Connector_Generic:Conn_01x04
Connections:
- net +3V3: now also J7.2 (Pin_2)
- net GND: now also J7.1 (Pin_1)
- net KBD_SCL: now also J7.4 (Pin_4)
- net KBD_SDA: now also J7.3 (Pin_3)
Other:
- moved on the sheet: SW1
Changed lines of the file:
@@
 EESchema Schematic File Version 5
-EELAYER 32 0
+EELAYER 33 0
 EELAYER END
 $Descr A4 11693 8268
@@
 NoConn ~ 1800 2200
 NoConn ~ 1800 1500
-NoConn ~ 6050 1650
+NoConn ~ 6050 1000
 NoConn ~ 9800 1400
 NoConn ~ 5150 4550
@@
 	5200 4550 5150 4550
 Wire Wire Line
-	5650 1750 5600 1750
-Wire Wire Line
-	6050 1850 6100 1850
-Wire Wire Line
-	6100 1850 6100 1900
+	5650 1100 5600 1100
+Wire Wire Line
+	5850 1900 5900 1900
+Wire Wire Line
+	5850 2000 5900 2000
+Wire Wire Line
+	5850 2100 5900 2100
+Wire Wire Line
+	5850 2200 5900 2200
+Wire Wire Line
+	6050 1200 6100 1200
+Wire Wire Line
+	6100 1200 6100 1250
 Wire Wire Line
 	6600 3450 6650 3450
@@
 Text Label 5150 4450 2    50   ~ 0
 TX
-Text Label 5600 1750 2    50   ~ 0
+Text Label 5600 1100 2    50   ~ 0
 EN
+Text Label 5900 2100 0    50   ~ 0
+SDA
+Text Label 5900 2200 0    50   ~ 0
+SCL
 Text Label 6650 3550 0    50   ~ 0
 EN
@@
 $EndComp
 $Comp
+L power:+3.3V #PWR?
+U 1 1 5E900AF8
+P 5900 2000
+F 0 "#PWR?" H 5900 1850 50  0001 C CNN
+F 1 "+3.3V" V 5900 2150 50  0000 L CNN
+F 2 "" H 5900 2000 50  0001 C CNN
+F 3 "" H 5900 2000 50  0001 C CNN
+	1    5900 2000
+	0    1    1    0
+$EndComp
+$Comp
 L power:+BATT #PWR05
 U 1 1 5CD3C192
@@
 $EndComp
 $Comp
+L power:GND #PWR?
+U 1 1 5E9010D0
+P 5900 1900
+F 0 "#PWR?" H 5900 1650 50  0001 C CNN
+F 1 "GND" V 5900 1750 50  0000 R CNN
+F 2 "" H 5900 1900 50  0001 C CNN
+F 3 "" H 5900 1900 50  0001 C CNN
+	1    5900 1900
+	0    -1   -1   0
+$EndComp
+$Comp
 L power:GND #PWR04
 U 1 1 5CDB1AC0
-P 6100 1900
-F 0 "#PWR04" H 6100 1650 50  0001 C CNN
-F 1 "GND" H 6105 1727 50  0000 C CNN
-F 2 "" H 6100 1900 50  0001 C CNN
-F 3 "" H 6100 1900 50  0001 C CNN
-	1    6100 1900
+P 6100 1250
+F 0 "#PWR04" H 6100 1000 50  0001 C CNN
+F 1 "GND" H 6105 1077 50  0000 C CNN
+F 2 "" H 6100 1250 50  0001 C CNN
+F 3 "" H 6100 1250 50  0001 C CNN
+	1    6100 1250
 	1    0    0    -1
 $EndComp
@@
 $EndComp
 $Comp
+L Connector_Generic:Conn_01x04 J7
+U 1 1 5E4ACB99
+P 5650 2000
+F 0 "J7" H 5650 2200 50  0000 C CNN
+F 1 "Conn_Stemma_QT" V 5750 1950 50  0000 C CNN
+F 2 "Connector_JST:JST_SH_SM04B-SRSS-TB_1x04-1MP_P1.00mm_Horizontal" H 5650 2000 50  0001 C CNN
+F 3 "~" H 5650 2000 50  0001 C CNN
+	1    5650 2000
+	-1   0    0    -1
+$EndComp
+$Comp
 L Switch:SW_SPDT SW1
 U 1 1 5CDAF66A
-P 5850 1750
-F 0 "SW1" H 5850 1943 50  0000 C CNN
-F 1 "SW_EN" H 5850 1944 50  0001 C CNN
-F 2 "Button_Switch_SMD:SW_SPDT_PCM12" H 5850 1750 50  0001 C CNN
-F 3 "~" H 5850 1750 50  0001 C CNN
-	1    5850 1750
-	1    0    0    -1
-$EndComp
+P 5850 1100
+F 0 "SW1" H 5850 1293 50  0000 C CNN
+F 1 "SW_EN" H 5850 1294 50  0001 C CNN
+F 2 "Button_Switch_SMD:SW_SPDT_PCM12" H 5850 1100 50  0001 C CNN
+F 3 "~" H 5850 1100 50  0001 C CNN
+	1    5850 1100
+	1    0    0    -1
+$EndComp
