File: keyboard.sch (KiCad schematic (older format))
At the start: 16 parts, among them Q1 BSS138, SW2 SW_RIGHT, SW3 SW_LEFT, U1 5-Way_Switch, U2 BBQ10KBD, U3 ATSAMD20E16A

Commit message: Finish up rev1
Parts:
- removed U3: ATSAMD20E16A, Package_DFN_QFN:QFN-32-1EP_5x5mm_P0.5mm_EP3.45x3.45mm, symbol MCU_Microchip_SAMD_Extra:ATSAMD20E16A
- added C11, C12: 0.1uF, Capacitor_SMD:C_0603_1608Metric, symbol Device:C_Small
- added SW4: SW_RIGHT2, Button_Switch_SMD_Extra:RMT-CZ66, symbol Switch:SW_SPST
- added SW5: SW_LEFT2, Button_Switch_SMD_Extra:RMT-CZ66, symbol Switch:SW_SPST
- added TP10: TP_KBD_GND, TestPoint:TestPoint_Pad_D3.0mm, symbol Connector:TestPoint
- added TP9: TP_KBD_3V, TestPoint:TestPoint_Pad_D3.0mm, symbol Connector:TestPoint
- added U7: ATSAMD20G16A, Package_DFN_QFN:QFN-48-1EP_7x7mm_P0.5mm_EP5.15x5.15mm, symbol MCU_Microchip_SAMD_Extra:ATSAMD20G16A
- SW2: value SW_RIGHT -> SW_RIGHT1; footprint (none) -> Button_Switch_SMD_Extra:RMT-CZ66
- SW3: value SW_LEFT -> SW_LEFT1; footprint (none) -> Button_Switch_SMD_Extra:RMT-CZ66
- U1: footprint (none) -> Button_Switch_SMD_Extra:SF303GJ26
- U2: footprint (none) -> Connector_Hirose_Extra:BM14B(0.8)-24DS-0.4V(53)
Connections:
- net +3V3: now also C11.1, C12.1, TP9.1, U7.17 (VDDIO), U7.36 (VDDIO), U7.44 (VDDIN), U7.6 (VDD)
- net BL_CTRL: now also U7.19 (PB10)
- net GND: now also C11.2, C12.2, SW4.1 (A), SW5.1 (A), TP10.1, U7.18 (GND), U7.35 (GND), U7.42 (GND), U7.5 (GND)
- net INT: now also U7.37 (PB22)
- net JOY_CENTER: now also U7.11 (PA06)
- net JOY_DOWN: now also U7.8 (PB09)
- net JOY_LEFT: now also U7.10 (PA05)
- net JOY_RIGHT: now also U7.9 (PA04)
- net JOY_UP: now also U7.12 (PA07)
- net KBD_COL1: now also U7.21 (PA12)
- net KBD_COL2: now also U7.23 (PA14)
- net KBD_COL3: now also U7.24 (PA15)
- net KBD_COL4: now also U7.25 (PA16)
- net KBD_COL5: now also U7.27 (PA18)
- net KBD_ROW1: now also U7.20 (PB11)
- net KBD_ROW2: now also U7.22 (PA13)
- net KBD_ROW3: now also U7.26 (PA17); no longer TP4.1
- net KBD_ROW4: now also U7.28 (PA19)
- net KBD_ROW5: now also U7.29 (PA20)
- net KBD_ROW6: now also U7.30 (PA21)
- net KBD_ROW7: now also U7.32 (PA23)
- net SCL: now also U7.14 (PA09)
- net SDA: now also U7.13 (PA08)
- net ~RESET~: now also U7.40 (~RESET~)
- net at C3.1: now also U7.43 (VDDCORE)
- net at R5.2, TP2.1: now also U7.45 (SWCLK)
- net at TP3.1: now also U7.46 (SWDIO)
- net BTN_LEFT renamed BTN_LEFT1
- net BTN_LEFT1: now also U7.1 (PA00)
- net BTN_RIGHT renamed BTN_RIGHT1
- net BTN_RIGHT1: now also U7.3 (PA02)
- new net: TP4.1, U7.31 (PA22)
- new net BTN_LEFT2: SW5.2 (B), U7.2 (PA01)
- new net BTN_RIGHT2: SW4.2 (B), U7.4 (PA03)
- no-connect marks 1 -> 10
Other:
- note added: "For SWD header"
- moved on the sheet: C1, C2, C3, R5, SW2, SW3, TP2, TP3, TP4
