File: lcd.sch (KiCad schematic (older format))
At the start: 7 parts, among them Q2 BSS138, U4 ER-TFT02X

Commit message: Finish up rev1
Parts:
- U4: footprint (none) -> Connector_EastRising:ER-CON50HT-1
Changed lines of the file:
@@
 F 0 "U4" H 6550 4850 60  0000 R CNN
 F 1 "ER-TFT02X" H 6100 1850 60  0000 C CNN
-F 2 "" H 6100 2650 60  0001 C CNN
+F 2 "Connector_EastRising:ER-CON50HT-1" H 6100 2650 60  0001 C CNN
 F 3 "" H 6100 2650 60  0001 C CNN
 	1    6100 3400
