File: keyboard_featherwing.kicad_pcb (KiCad board)
At the start: 2 copper layers, 68 x 100 mm, 58 parts, among them J3 Micro_SD_Card_Det, J7 Conn_Stemma_QT, Q1 BSS138, Q2 BSS138, SW1 SW_EN, SW2 SW_RIGHT1, SW3 SW_LEFT1, SW4 SW_RIGHT2, SW5 SW_LEFT2, U1 5-Way_Switch, U2 BBQ10KBD, U4 ER-TFT02X, U5 STMPE811, U6 Adafruit_Feather_2X, U7 ATSAMD20G16A, U8 74AHCT1G125

Commit message: Rev5, production
Other:
- net class Default removed
- board text added: "Keyboard FeatherWing by arturo182 April 2020"
- board text removed: "Keyboard FeatherWing by arturo182 March 2020"
- board text removed: "Remember to order 1.2mm!"
